File: G0-022M6.kicad_sch (KiCad schematic)
At the start: 30 parts, among them J1 SolderJumper_3_Open, J10 Solder Pad, J11 Conn_01x04, J2 SolderJumper_2_Open, J3 SolderJumper_2_Open, J4 SolderJumper_2_Open, J5 Game_Edge_Connector, J6 Cart_Edge_Connector, J7 Solder Pad, J8 Solder Pad, J9 Solder Pad, Q1 Unknown, Q2 Unknown, U1 Front FFEATX001, U2 W29C020, U3 Unknown DIP32, U4 Unknown TSOP32

Commit message: Add files via upload
Parts:
- C1, C2, C4: value C_Small -> 100 nF
- C3, C5: value C_Small -> Unknown
- C6: value C_Polarized_Small_US -> Unknown
- R1, R2: value R_Small_US -> 4.7K Ohm
- R3, R4, R6: value R_Small_US -> Unknown
- R5: value R_Small_US -> 220K Ohm
Changed lines of the file:
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@@
       (effects (font (size 1.27 1.27)) (justify left))
     )
-    (property "Value" "C_Small" (at 223.52 131.4513 0)
+    (property "Value" "100 nF" (at 223.52 131.4513 0)
       (effects (font (size 1.27 1.27)) (justify left))
     )
@@
       (effects (font (size 1.27 1.27)) (justify left))
     )
-    (property "Value" "C_Small" (at 175.26 131.4513 0)
+    (property "Value" "100 nF" (at 175.26 131.4513 0)
       (effects (font (size 1.27 1.27)) (justify left))
     )
@@
       (effects (font (size 1.27 1.27)) (justify left))
     )
-    (property "Value" "C_Small" (at 238.76 131.4513 0)
+    (property "Value" "Unknown" (at 238.76 131.4513 0)
       (effects (font (size 1.27 1.27)) (justify left))
     )
@@
       (effects (font (size 1.27 1.27)) (justify left))
     )
-    (property "Value" "R_Small_US" (at 218.44 155.575 0)
+    (property "Value" "Unknown" (at 218.44 155.575 0)
       (effects (font (size 1.27 1.27)) (justify left))
     )
@@
       (effects (font (size 1.27 1.27)) (justify left))
     )
-    (property "Value" "R_Small_US" (at 267.97 155.575 0)
+    (property "Value" "Unknown" (at 267.97 155.575 0)
       (effects (font (size 1.27 1.27)) (justify left))
     )
@@
       (effects (font (size 1.27 1.27)) (justify left))
     )
-    (property "Value" "R_Small_US" (at 201.93 155.575 0)
+    (property "Value" "4.7K Ohm" (at 201.93 155.575 0)
       (effects (font (size 1.27 1.27)) (justify left))
     )
@@
       (effects (font (size 1.27 1.27)) (justify left))
     )
-    (property "Value" "C_Small" (at 208.28 131.4513 0)
+    (property "Value" "Unknown" (at 208.28 131.4513 0)
       (effects (font (size 1.27 1.27)) (justify left))
     )
@@
       (effects (font (size 1.27 1.27)) (justify left))
     )
-    (property "Value" "R_Small_US" (at 185.42 155.575 0)
+    (property "Value" "4.7K Ohm" (at 185.42 155.575 0)
       (effects (font (size 1.27 1.27)) (justify left))
     )
@@
       (effects (font (size 1.27 1.27)) (justify left))
     )
-    (property "Value" "R_Small_US" (at 234.95 155.575 0)
+    (property "Value" "Unknown" (at 234.95 155.575 0)
       (effects (font (size 1.27 1.27)) (justify left))
     )
@@
       (effects (font (size 1.27 1.27)) (justify left))
     )
-    (property "Value" "R_Small_US" (at 251.46 155.575 0)
+    (property "Value" "220K Ohm" (at 251.46 155.575 0)
       (effects (font (size 1.27 1.27)) (justify left))
     )
@@
       (effects (font (size 1.27 1.27)) (justify left))
     )
-    (property "Value" "C_Polarized_Small_US" (at 255.27 131.0132 0)
+    (property "Value" "Unknown" (at 255.27 131.0132 0)
       (effects (font (size 1.27 1.27)) (justify left))
     )
@@
       (effects (font (size 1.27 1.27)) (justify left))
     )
-    (property "Value" "C_Small" (at 193.04 131.4513 0)
-      (effects (font (size 1.27 1.27)) (justify left))
-    )
+    (property "Value" "100 nF" (at 193.04 131.4513 0)
+      (effects (font (size 1.27 1.27)) (justify left))
+    )
